File: hardware/kikard.kicad_sch (KiCad schematic)
At the start: 1 part, among them U1 NRF52840-QIAA-R

Commit message: 6-4-25
Parts:
- added J1: USB_C_Receptacle_USB2.0_16P, symbol Connector:USB_C_Receptacle_USB2.0_16P
- added R1, R2: 5.1k, symbol Device:R
- added U2: ST25R3916-AQWT, ST25R3916-AQWT:QFN50P500X500X100-33N, symbol ST25R3916-AQWT:ST25R3916-AQWT
Connections:
- net vbus: now reaches U1.AD2 (VBUS)
- net vbus: now also J1.A4 (VBUS), J1.A9 (VBUS), J1.B4 (VBUS), J1.B9 (VBUS)
- net D-: now reaches U1.AD4 (D-)
- net D-: now also J1.A7 (D-), J1.B7 (D-)
- net D+: now reaches U1.AD6 (D+)
- net D+: now also J1.A6 (D+), J1.B6 (D+)
- new net: J1.A5 (CC1), R1.1
- new net: J1.B5 (CC2), R2.1
- new net: U2.12 (GND_DR), U2.16 (GND_DR)
- new net GND: J1.A1 (GND), J1.A12 (GND), J1.B1 (GND), J1.B12 (GND), R1.2, R2.2

Commit message: 6-6-25
Parts:
- added C1, C2, C3: 4.7uF, symbol Device:C
- added C10, C12, C14, C16, C18, C4, C6, C8: 10nF, symbol Device:C
- added C11: 1uF, symbol Device:C
- added C13, C15, C17, C19, C5, C7, C9: 2.2uF, symbol Device:C
- added C20, C21: 6pF, symbol Device:C
- added Y1: XRCGB27M120F3M00R0, symbol Device:Crystal_GND2
Connections:
- net vbus is gone; now on net vusb: J1.A4 (VBUS), J1.A9 (VBUS), J1.B4 (VBUS), J1.B9 (VBUS), U1.AD2 (VBUS)
- net GND: now also J1.S1 (SHIELD), U1.74 (VSS), U1.B7 (VSS), U2.12 (GND_DR), U2.16 (GND_DR), U2.20 (I2C_EN), U2.21 (VSS), U2.26 (GND_A), U2.33 (EXP), U2.6 (GND_D), C1.1, C10.1, C11.1, C12.1, C13.1, C14.1, C15.1, C16.1, C17.1, C18.1, C19.1, C2.1, C20.1, C21.1, C3.2, C4.1, C5.1, C6.1, C7.1, C8.1, C9.1, Y1.2
- net VDD3.3v: now reaches U2.1 (VDD_IO)
- net VDD3.3v: now also U1.A22 (VDD), U1.AD14 (VDD), U1.AD23 (VDD), U1.B1 (VDD), U1.W1 (VDD), C2.2, C6.2, C7.2
- net vusb: now reaches U2.10 (VDD_TX)
- net vusb: now also U2.8 (VDD), C3.1, C4.2, C5.2, C8.2, C9.2
- net at U2.11 (VDD_AM): now also C14.2, C15.2
- net at U2.14 (VDD_DR): now also U2.9 (VDD_RF), C12.2, C13.2
- net at U2.24 (AGDC): now also C10.2, C11.2
- net IRQ: now reaches U2.27 (IRQ)
- net IRQ: now also U1.N1 (P0.08)
- net CS: now reaches U2.29 (~{BSS})
- net CS: now also U1.M2 (P0.07/TRACECLK)
- net at U2.3 (VDD_D): now also C18.2, C19.2
- net SCLK: now reaches U2.30 (SCLK/SCL)
- net SCLK: now also U1.J1 (P0.04/AIN2)
- net MOSI: now reaches U2.31 (MOSI)
- net MOSI: now also U1.K2 (P0.05/AIN3)
- net MISO: now reaches U2.32 (MISO/SDA)
- net MISO: now also U1.L1 (P0.06)
- net at U2.4 (XTO): now also C21.2, Y1.3
- net at U2.5 (XTI): now also C20.2, Y1.1
- net at U2.7 (VDD_A): now also C16.2, C17.2
- net at U1.AC5 (DECUSB): now also C1.2
Other:
- moved on the sheet: U2

Commit message: 6-29-25
Parts:
- added AE1: Texas_SWRA117D_2.4GHz_Right, extra-symbols-footprints:Texas_SWRA117D_2.4GHz_Right, symbol Device:Antenna_Chip
- added C22, C23: 12pF, symbol Device:C
- added C24, C25: 6pF, symbol Device:C
- added C26: 47nF, symbol Device:C
- added C27: 1uF, symbol Device:C
- added C28, C29, C30, C31: 100nF, symbol Device:C
- added C32: 4.7uF, symbol Device:C
- added C33: 0.8pF, symbol Device:C
- added L1: 10uH, symbol Device:L
- added L2: 15nH, symbol Device:L
- added L3: 3.9nH, symbol Device:L
- added Y2: X201632MOB4SI, symbol Device:Crystal_GND24
- added Y3: X161032768KGD2SI, symbol Device:Crystal
Connections:
- net GND: now also U1.F23 (VSS_PA), AE1.1 (FEED), C22.2, C23.2, C24.1, C25.1, C26.1, C27.1, C28.2, C29.2, C30.1, C31.1, C32.1, C33.1, Y2.2, Y2.4
- net VDD3.3v: now also U1.Y2 (VDDH), C30.2, C31.2; no longer U1.B1 (VDD)
- net at U1.A23 (XC2): now also C22.1, Y2.3
- net at U1.B24 (XC1): now also C23.1, Y2.1
- net at U1.B3 (DCC): now also L1.1
- net DCC: now reaches U1.B5 (DEC4)
- net DCC: now also U1.E24 (DEC6), C26.2, C27.2, L2.2
- net at U1.C1 (DEC1): now also C29.1
- net at U1.D2 (P0.00/XL1): now also C24.2, Y3.2
- net at U1.D23 (DEC3): now also C28.1
- net at U1.F2 (P0.01/XL2): now also C25.2, Y3.1
- net at U1.H23 (ANT): now also C33.2, L3.2
- new net: C32.2, U1.B1 (VDD)
- new net: AE1.2 (PCB_Trace), L3.1
- new net: L1.2, L2.1
Other:
- moved on the sheet: C1, C2, C3

Commit message: 7-9-25
Parts:
- added AE2: Antenna_Loop, extra-symbols-footprints:kikard-ant-v1.0, symbol Device:Antenna_Loop
- added C34: 100nF, symbol Device:C
Connections:
- net GND: now also C34.1
- net VDD3.3v: now also C32.2, U1.B1 (VDD), C34.2

Commit message: 7-11-25
Parts:
- added C35, C37, C41, C44: 100pF, symbol Device:C
- added C36, C43: 10pF, symbol Device:C
- added C38, C40: 680pF, symbol Device:C
- added C39, C42: 62pF, symbol Device:C
- added C45, C46: 1nF NP0, symbol Device:C
- added L4, L5: 270uH, symbol Device:L
- added Q1, Q2: WNM3013-3/TR, extra-symbols-footprints:SOT-723_L1.2-W0.8-P0.40-LS1.2-BR, symbol WNM3013-3TR:WNM3013-3_TR
- added R3, R4: 100K, symbol Device:R
Connections:
- net CS: now also U1.AD20 (P0.24); no longer U1.M2 (P0.07/TRACECLK)
- net GND: now also C35.2, C38.1, C39.1, C40.2, C42.2, C44.1, R3.1, R4.1
- net IRQ: now also U1.AC21 (P0.25); no longer U1.N1 (P0.08)
- net MISO: now also U1.AC19 (P0.23); no longer U1.L1 (P0.06)
- net MOSI: now also U1.AD18 (P0.22); no longer U1.K2 (P0.05/AIN3)
- net SCLK: now also U1.AC17 (P0.21); no longer U1.J1 (P0.04/AIN2)
- net ST_RFO1: now reaches U2.13 (RFO1)
- net ST_RFO1: now also L4.2
- net ST_RFO2: now reaches U2.15 (RFO2)
- net ST_RFO2: now also L5.2
- net ST_RFI1: now reaches U2.22 (RFI1)
- net ST_RFI1: now also C35.1, C36.2
- net ST_RFI2: now reaches U2.23 (RFI2)
- net ST_RFI2: now also C43.2, C44.2
- net NRF_NFC_2: now reaches U1.J24 (P0.10/NFC2)
- net NRF_NFC_2: now also Q2.2 (S), R4.2
- net NRF_NFC_1: now reaches U1.L24 (P0.09/NFC1)
- net NRF_NFC_1: now also Q1.2 (S), R3.2
- net NFC_ANT_1: now reaches AE2.1
- net NFC_ANT_1: now also C36.1, C37.1, C39.2, C45.1
- net NFC_ANT_2: now reaches AE2.2
- net NFC_ANT_2: now also C41.1, C42.1, C43.1, C46.1
- new net: C40.1, C41.2, L5.1
- new net: C45.2, Q1.3 (D)
- new net: C37.2, C38.2, L4.1
- new net: C46.2, Q2.3 (D)
- new net NFC_SW: Q1.1 (G), Q2.1 (G), U1.N1 (P0.08)

Commit message: 7-14-25
Parts:
- removed J1: USB_C_Receptacle_USB2.0_16P, symbol Connector:USB_C_Receptacle_USB2.0_16P
- added C47: 100nF, extra-symbols-footprints:C0402, symbol Device:C
- added LED1, LED2: WS2812B-2020, extra-symbols-footprints:LED-SMD_4P-L2.0-W2.0-TL_WS2812B-2020, symbol WS2812B-2020:WS2812B-2020
- added R5: 10k, extra-symbols-footprints:R0402, symbol Device:R
- added SW1, SW2, SW3: K2-6639SP-C4SC-04, extra-symbols-footprints:KEY-SMD_4P-L6.0-W6.0-P3.90-LS9.0, symbol K2-6639SP-C4SC-04:K2-6639SP-C4SC-04
- added SW4: HX TS-1088-AR02016, extra-symbols-footprints:SW-SMD_L4.0-W2.9-LS5.0, symbol HX3x4x2-2P-2.5N:HXTS-1088-AR02016
- added USB1: TYPE-C16PIN, extra-symbols-footprints:USB-C-SMD_TYPE-C16PIN, symbol USB-C:TYPE-C16PIN
- C1, C13, C15, C17, C19, C2, C3, C32, C5, C7, C9: footprint (none) -> extra-symbols-footprints:C0603
- C10, C11, C12, C14, C16, C18, C20, C21, C22, C23, C24, C25, C26, C27, C28, C29, C30, C31, C33, C34, C35, C36, C37, C38, C39, C4, C40, C41, C42, C43, C44, C6, C8: footprint (none) -> extra-symbols-footprints:C0402
- C45, C46: value 1nF NP0 -> 1nF; footprint (none) -> extra-symbols-footprints:C0402
- L1, L2: footprint (none) -> extra-symbols-footprints:L0603
- L3, R1, R2: footprint (none) -> extra-symbols-footprints:R0402
- L4, L5: value 270uH -> 270nH; footprint (none) -> extra-symbols-footprints:L0402
- R3, R4: footprint (none) -> extra-symbols-footprints:R0603
- Y1: value XRCGB27M120F3M00R0 -> 27MHz; footprint (none) -> extra-symbols-footprints:CRYSTAL-SMD_4P-L2.0-W1.6-BL-B
- Y2: value X201632MOB4SI -> 32MHz; footprint (none) -> extra-symbols-footprints:CRYSTAL-SMD_4P-L2.0-W1.6-BL-2
- Y3: value X161032768KGD2SI -> 32.768kHz; footprint (none) -> extra-symbols-footprints:OSC-SMD_L1.6-W1.0
Connections:
- net D+: now also USB1.A6 (DP1), USB1.B6 (DP2)
- net D-: now also USB1.A7 (DN1), USB1.B7 (DN2)
- net GND: now also C47.2, LED1.2 (GND), LED2.2 (GND), SW1.3, SW1.4, SW2.3, SW2.4, SW3.3, SW3.4, SW4.2, USB1.1 (SHELL), USB1.2 (SHELL), USB1.3 (SHELL), USB1.4 (SHELL), USB1.A1B12 (GND), USB1.B1A12 (GND)
- net VDD3.3v: now also R5.1
- net vusb: now also LED1.4 (VDD), LED2.4 (VDD), USB1.A4B9 (VBUS), USB1.B4A9 (VBUS)
- net at R1.1: now also USB1.A5 (CC1)
- net at R2.1: now also USB1.B5 (CC2)
- net RESET: now reaches U1.AC13 (P0.18/NRESET)
- net RESET: now also C47.1, R5.2, SW4.1
- net BUTTON_3: now reaches U1.P23 (P1.07)
- net BUTTON_3: now also SW3.1, SW3.2
- net BUTTON_2: now reaches U1.R24 (P1.06)
- net BUTTON_2: now also SW2.1, SW2.2
- net BUTTON_1: now reaches U1.T23 (P1.05)
- net BUTTON_1: now also SW1.1, SW1.2
- net NEOPIXEL_2: now reaches U1.W24 (P1.02)
- net NEOPIXEL_2: now also LED2.3 (DI)
- net NEOPIXEL_1: now reaches U1.Y23 (P1.01)
- net NEOPIXEL_1: now also LED1.3 (DI)
Other:
- moved on the sheet: C39, C42, R1, R2

Commit message: 7-16-25
Parts:
- U1: footprint NRF52840-QIAA-R:XCVR_NRF52840-QIAA-R -> extra-symbols-footprints:XCVR_NRF52840-QIAA-R
- U2: footprint ST25R3916-AQWT:QFN50P500X500X100-33N -> extra-symbols-footprints:QFN50P500X500X100-33N
Changed lines of the file:
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@@
 			)
 		)
-		(property "Footprint" "ST25R3916-AQWT:QFN50P500X500X100-33N"
+		(property "Footprint" "extra-symbols-footprints:QFN50P500X500X100-33N"
 			(at 402.59 455.93 0)
 			(effects
@@
 			)
 		)
-		(property "Footprint" "NRF52840-QIAA-R:XCVR_NRF52840-QIAA-R"
+		(property "Footprint" "extra-symbols-footprints:XCVR_NRF52840-QIAA-R"
 			(at 182.88 441.96 0)
 			(effects

Commit message: 7-17-25
Connections:
- net CS: now also U1.AC11 (P0.16); no longer U1.AD20 (P0.24)
- net GND: now also U1.74_1 (VSS); no longer U1.74 (VSS)
- net MOSI: now also U1.AC9 (P0.14); no longer U1.AD18 (P0.22)
- net NEOPIXEL_1: now also U1.AD8 (P0.13); no longer U1.Y23 (P1.01)
Changed lines of the file:
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@@
 	(global_label "MOSI"
 		(shape input)
-		(at 154.94 464.82 180)
+		(at 154.94 444.5 180)
 		(fields_autoplaced yes)
 		(effects
@@
 		)
 		(property "Intersheetrefs" "${INTERSHEET_REFS}"
-			(at 147.3586 464.82 0)
+			(at 147.3586 444.5 0)
 			(effects
 				(font
@@
 	(global_label "NEOPIXEL_1"
 		(shape input)
-		(at 210.82 431.8 0)
+		(at 154.94 441.96 180)
 		(fields_autoplaced yes)
 		(effects
@@
 				(size 1.27 1.27)
 			)
-			(justify left)
+			(justify right)
 		)
 		(property "Intersheetrefs" "${INTERSHEET_REFS}"
-			(at 225.0537 431.8 0)
+			(at 140.7063 441.96 0)
 			(effects
 				(font
 					(size 1.27 1.27)
 				)
-				(justify left)
+				(justify right)
 				(hide yes)
 			)
@@
 	(global_label "CS"
 		(shape input)
-		(at 154.94 469.9 180)
+		(at 154.94 449.58 180)
 		(fields_autoplaced yes)
 		(effects
@@
 		)
 		(property "Intersheetrefs" "${INTERSHEET_REFS}"
-			(at 149.4753 469.9 0)
+			(at 149.4753 449.58 0)
 			(effects
 				(font
@@
 		(pin "A14"
 		)
-		(pin "74"
+		(pin "74_1"
 		)
 		(pin "G1"
