File: hardware/kikard.kicad_sch (KiCad schematic)
At the start: 73 parts, among them Q1 WNM3013-3/TR, Q2 WNM3013-3/TR, SW1 K2-6639SP-C4SC-04, SW2 K2-6639SP-C4SC-04, SW3 K2-6639SP-C4SC-04, SW4 HX TS-1088-AR02016, U1 NRF52840-QIAA-R, U2 ST25R3916-AQWT, Y1 27MHz, Y2 32MHz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

Commit message: 7-18-25
Parts:
- removed Y1: 27MHz, extra-symbols-footprints:CRYSTAL-SMD_4P-L2.0-W1.6-BL-B, symbol Device:Crystal_GND2
- added Y1: 27MHz, extra-symbols-footprints:CRYSTAL-SMD_4P-L2.0-W1.6-BL-B, symbol Device:Crystal_GND24
- L3: footprint extra-symbols-footprints:R0402 -> extra-symbols-footprints:L0402
- LED1, LED2: value WS2812B-2020 -> ZSRGB-2017H-08-Z3; footprint extra-symbols-footprints:LED-SMD_4P-L2.0-W2.0-TL_WS2812B-2020 -> extra-symbols-footprints:LED-SMD_4P-L2.0-W1.8-P0.90_XGM-S0807RGB; symbol WS2812B-2020:WS2812B-2020 -> rgbled:ZSRGB-2017H-08-Z3; LCSC Part C965555 -> C7497245
Connections:
- net GND: now also LED1.4 (GND), LED2.4 (GND), U1.74 (VSS), Y1.1, Y1.3; no longer U1.74_1 (VSS)
- net IRQ: now also U1.AC9 (P0.14); no longer U1.AC21 (P0.25)
- net MISO: now also U1.AC21 (P0.25); no longer U1.AC19 (P0.23)
- net MOSI: now also U1.AC19 (P0.23); no longer U1.AC9 (P0.14)
- net vusb: now also LED1.1 (VDD), LED2.1 (VDD); no longer LED1.4 (VDD), LED2.4 (VDD)
- net at C20.2, U2.5 (XTI): now also Y1.2
- net at C21.2, U2.4 (XTO): now also Y1.4

Commit message: 7-25-25
Parts:
- added TP1, TP2, TP3, TP4, TP5: TestPoint, extra-symbols-footprints:TestPoint_Pad_D1.0mm, symbol Connector:TestPoint
Connections:
- net GND: now also TP4.1
- net RESET: now also TP5.1
- net VDD3.3v: now also TP3.1
- net at U1.AA24 (SWDCLK): now also TP1.1
- net at U1.AC24 (SWDIO): now also TP2.1

Commit message: Fix BLE ant
Connections:
- net GND: now also AE1.2 (PCB_Trace); no longer AE1.1 (FEED)
- net at L3.1: now also AE1.1 (FEED); no longer AE1.2 (PCB_Trace)
Changed lines of the file:
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@@
 	(wire
 		(pts
-			(xy 226.06 458.47) (xy 251.46 458.47)
-		)
-		(stroke
-			(width 0)
-			(type default)
-		)
-	)
-	(wire
-		(pts
 			(xy 236.22 491.49) (xy 254 491.49)
 		)
@@
 	(wire
 		(pts
-			(xy 251.46 458.47) (xy 251.46 444.5)
-		)
-		(stroke
-			(width 0)
-			(type default)
-		)
-	)
-	(wire
-		(pts
 			(xy 254 482.6) (xy 254 476.25)
 		)
@@
 	(wire
 		(pts
+			(xy 226.06 458.47) (xy 246.38 458.47)
+		)
+		(stroke
+			(width 0)
+			(type default)
+		)
+	)
+	(wire
+		(pts
 			(xy 407.67 496.57) (xy 426.72 496.57)
 		)
@@
 	(wire
 		(pts
+			(xy 246.38 458.47) (xy 246.38 444.5)
+		)
+		(stroke
+			(width 0)
+			(type default)
+		)
+	)
+	(wire
+		(pts
 			(xy 422.91 478.79) (xy 426.72 478.79)
 		)
@@
 	(symbol
 		(lib_id "power:GND")
-		(at 246.38 444.5 0)
+		(at 251.46 444.5 0)
 		(unit 1)
 		(exclude_from_sim no)
@@
 		(fields_autoplaced yes)
 		(property "Reference" "#PWR026"
-			(at 246.38 450.85 0)
+			(at 251.46 450.85 0)
 			(effects
 				(font
@@
 		)
 		(property "Value" "GND"
-			(at 246.38 449.58 0)
+			(at 251.46 449.58 0)
 			(effects
 				(font
@@
 		)
 		(property "Footprint" ""
-			(at 246.38 444.5 0)
+			(at 251.46 444.5 0)
 			(effects
 				(font
@@
 		)
 		(property "Datasheet" ""
-			(at 246.38 444.5 0)
+			(at 251.46 444.5 0)
 			(effects
 				(font
@@
 		)
 		(property "Description" "Power symbol creates a global label with name \"GND\" , ground"
-			(at 246.38 444.5 0)
+			(at 251.46 444.5 0)
 			(effects
 				(font
