File: hardware/kikard.kicad_pcb (KiCad board)
At the start: 2 copper layers, 40 x 70 mm, 73 parts, among them Q1 WNM3013-3/TR, Q2 WNM3013-3/TR, SW1 K2-6639SP-C4SC-04, SW2 K2-6639SP-C4SC-04, SW3 K2-6639SP-C4SC-04, SW4 HX TS-1088-AR02016, U1 NRF52840-QIAA-R, U2 ST25R3916-AQWT, Y1 27MHz, Y2 32MHz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

Commit message: 7-17-25
Parts:
- moved C23 91.1 mm to (228.0, 126.0), turned to -90 degrees
- moved C33 85.8 mm to (225.9, 132.0), turned to 180 degrees
- moved C22 85.5 mm to (222.4, 122.0), turned to 180 degrees
- moved C47 84.7 mm to (230.0, 139.5)
- moved C30 82.6 mm to (222.0, 133.9), turned to 90 degrees
- moved C24 78.2 mm to (213.4, 141.0), turned to 180 degrees
- moved C25 77.5 mm to (213.4, 139.5), turned to 180 degrees
- moved C28 75.1 mm to (215.4, 120.5), turned to 180 degrees
- moved C29 73.0 mm to (212.0, 132.9), turned to -90 degrees
- moved C26 72.5 mm to (209.5, 127.5), turned to -90 degrees
- moved C27 71.8 mm to (211.0, 127.5), turned to -90 degrees
- moved C1 65.4 mm to (213.5, 134.3), turned to 90 degrees
- moved Y3 60.4 mm to (211.5, 137.5), turned to 180 degrees
- moved C31 59.7 mm to (220.5, 133.9), turned to 90 degrees
- moved LED2 58.3 mm to (226.9, 145.1), turned to 90 degrees
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Connections:
- U1 pad 74: GND -> (no net)
- U1 pad 74_1: (no net) -> GND
- U1 pad AC11: unconnected-(U1-P0.16-PadAC11) -> CS
- U1 pad AC9: unconnected-(U1-P0.14-PadAC9) -> MOSI
- U1 pad AD18: MOSI -> unconnected-(U1-P0.22-PadAD18)
- U1 pad AD20: CS -> unconnected-(U1-P0.24-PadAD20)
- U1 pad AD8: unconnected-(U1-P0.13-PadAD8) -> NEOPIXEL_1
- U1 pad Y23: NEOPIXEL_1 -> unconnected-(U1-P1.01-PadY23)
Routing:
- net GND: track 88.2 -> 179.3 mm, vias 0 -> 5
- net Net-(U1-ANT): track 0.00 -> 35.6 mm, vias 0 -> 4
- net RESET: track 0.00 -> 26.2 mm, vias 0 -> 2
- net DCC: track 0.00 -> 25.1 mm, vias 0 -> 4
- net VDD3.3v: track 26.6 -> 51.4 mm, vias 0 -> 3
- net Net-(U1-P0.00/XL1): track 0.00 -> 19.7 mm, vias 0 -> 2
- net vusb: track 20.8 -> 38.7 mm, vias 3 -> 5
- net NEOPIXEL_1: track 0.00 -> 16.9 mm, vias 0 -> 2
- net NEOPIXEL_2: track 0.00 -> 16.8 mm, vias 0 -> 2
- net Net-(U1-P0.01/XL2): track 0.00 -> 16.2 mm, vias 0 -> 2
- net Net-(U1-DEC3): track 0.00 -> 10.0 mm, vias 0 -> 2
- net Net-(U1-DEC1): track 0.00 -> 9.39 mm, vias 0 -> 2
- net Net-(U1-XC2): track 0.00 -> 9.36 mm
- net Net-(U1-XC1): track 0.00 -> 8.52 mm, vias 0 -> 2
- net Net-(U1-DECUSB): track 0.00 -> 6.19 mm, vias 0 -> 2
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
Commit message: 7-18-25
Parts:
- added G***: LOGO, extra-symbols-footprints:logo, F.Cu at (150.0, 78.5)
- added REF**: MountingHole_2.5mm_Pad, extra-symbols-footprints:MountingHole_2.5mm_Pad, F.Cu at (167.0, 132.0)
- added REF**: MountingHole_2.5mm_Pad, extra-symbols-footprints:MountingHole_2.5mm_Pad, F.Cu at (133.0, 68.0)
- added REF**: MountingHole_2.5mm_Pad, extra-symbols-footprints:MountingHole_2.5mm_Pad, F.Cu at (167.0, 68.0)
- added REF**: MountingHole_2.5mm_Pad, extra-symbols-footprints:MountingHole_2.5mm_Pad, F.Cu at (133.0, 132.0)
- L3: footprint extra-symbols-footprints:R0402 -> extra-symbols-footprints:L0402
- LED1, LED2: value WS2812B-2020 -> ZSRGB-2017H-08-Z3; footprint extra-symbols-footprints:LED-SMD_4P-L2.0-W2.0-TL_WS2812B-2020 -> extra-symbols-footprints:LED-SMD_4P-L2.0-W1.8-P0.90_XGM-S0807RGB
- moved AE1 73.5 mm to (135.6, 125.0)
- moved L3 72.9 mm to (138.6, 129.0)
- moved SW4 72.4 mm to (161.5, 129.0)
- moved U2 72.1 mm to (148.8, 100.4)
- moved AE2 71.6 mm to (137.5, 66.0)
- moved C1 71.6 mm to (143.5, 119.3)
- moved C2 71.6 mm to (145.5, 119.3)
- moved C22 71.6 mm to (152.4, 107.0)
- moved C23 71.6 mm to (158.0, 111.0)
- moved C24 71.6 mm to (143.4, 126.0)
- moved C25 71.6 mm to (143.4, 124.5)
- moved C26 71.6 mm to (139.5, 112.5)
- moved C27 71.6 mm to (141.0, 112.5)
- moved C28 71.6 mm to (145.4, 105.5)
- moved C29 71.6 mm to (142.0, 118.0)
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Connections:
- LED1 pad 1: unconnected-(LED1-DO-Pad1) -> vusb
- LED1 pad 4: vusb -> GND
- LED2 pad 1: unconnected-(LED2-DO-Pad1) -> vusb
- LED2 pad 4: vusb -> GND
- U1 pad 74: (no net) -> GND
- U1 pad AC19: MISO -> MOSI
- U1 pad AC21: IRQ -> MISO
- U1 pad AC9: MOSI -> IRQ
- Y1 pad 1: Net-(U2-XTI) -> GND
- Y1 pad 2: GND -> Net-(U2-XTI)
- Y1 pad 3: Net-(U2-XTO) -> GND
- Y1 pad 4: (no net) -> Net-(U2-XTO)
Routing:
- net GND: track 179.3 -> 324.6 mm, vias 5 -> 15
- net vusb: track 38.7 -> 90.0 mm, vias 5 -> 9
- net NRF_NFC_2: track 2.86 -> 45.0 mm, vias 1 -> 2
- net NRF_NFC_1: track 3.74 -> 44.3 mm, vias 1 -> 2
- net NFC_ANT_2: track 0.00 -> 39.1 mm, vias 0 -> 3
- net NFC_ANT_1: track 0.00 -> 29.7 mm, vias 0 -> 1
- net NFC_SW: track 0.00 -> 21.4 mm, vias 0 -> 4
- net ST_RFI2: track 0.00 -> 20.5 mm, vias 0 -> 2
- net Net-(U2-XTI): track 0.00 -> 16.8 mm, vias 0 -> 2
- net ST_RFI1: track 0.00 -> 16.3 mm
- net Net-(U2-XTO): track 0.00 -> 15.1 mm, vias 0 -> 2
- net MISO: track 0.00 -> 14.0 mm, vias 0 -> 2
- net SCLK: track 0.00 -> 13.8 mm, vias 0 -> 2
- net MOSI: track 0.00 -> 13.8 mm, vias 0 -> 2
- net CS: track 0.00 -> 13.2 mm, vias 0 -> 2
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Other:
- board text added: "KiKard"
- board text added: "m5kro"

Commit message: 7-25-25
Parts:
- added 3V3: TestPoint, extra-symbols-footprints:TestPoint_Pad_D1.0mm, F.Cu at (158.5, 119.0)
- added GND: TestPoint, extra-symbols-footprints:TestPoint_Pad_D1.0mm, F.Cu at (162.0, 119.0)
- added RST: TestPoint, extra-symbols-footprints:TestPoint_Pad_D1.0mm, F.Cu at (162.0, 122.5)
- added SCK: TestPoint, extra-symbols-footprints:TestPoint_Pad_D1.0mm, F.Cu at (158.5, 115.5)
- added SWD: TestPoint, extra-symbols-footprints:TestPoint_Pad_D1.0mm, F.Cu at (162.0, 115.5)
Connections:
- U1 pad AA24: unconnected-(U1-SWDCLK-PadAA24) -> Net-(U1-SWDCLK)
- U1 pad AC24: unconnected-(U1-SWDIO-PadAC24) -> Net-(U1-SWDIO)
Routing:
- net GND: track 324.6 -> 337.1 mm, vias 15 -> 17
- net Net-(U1-SWDIO): track 0.00 -> 11.7 mm, vias 0 -> 2
- net VDD3.3v: track 63.4 -> 73.1 mm, vias 5 -> 6
- net Net-(U1-SWDCLK): track 0.00 -> 5.86 mm, vias 0 -> 2
- net RESET: track 24.5 -> 27.9 mm

Commit message: Fix BLE ant
Parts:
- moved L3 2.00 mm to (138.4, 127.0)
- renumbered SCK to TP1, SWD to TP2, 3V3 to TP3, GND to TP4, RST to TP5
Connections:
- AE1 pad 1: GND -> Net-(AE1-FEED)
- AE1 pad 2: Net-(AE1-PCB_Trace) -> GND
- L3 pad 1: Net-(AE1-PCB_Trace) -> Net-(AE1-FEED)
Routing:
- net Net-(AE1-PCB_Trace): track 3.28 -> 0.00 mm
- net Net-(AE1-FEED): track 0.00 -> 3.08 mm
- net GND: track 337.1 -> 335.5 mm
- net Net-(U1-ANT): track 35.5 -> 36.3 mm
Changed lines of the file:
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@@
 	)
 	(net 0 "")
-	(net 1 "Net-(AE1-PCB_Trace)")
+	(net 1 "Net-(AE1-FEED)")
 	(net 2 "GND")
 	(net 3 "NFC_ANT_1")
@@
 		(descr "SMD pad as test Point, diameter 1.0mm")
 		(tags "test point SMD pad")
-		(property "Reference" "3V3"
+		(property "Reference" "TP3"
 			(at 0 -1.5 0)
 			(layer "F.SilkS")
@@
 		(descr "SMD pad as test Point, diameter 1.0mm")
 		(tags "test point SMD pad")
-		(property "Reference" "RST"
+		(property "Reference" "TP5"
 			(at 0 -1.448 0)
 			(layer "F.SilkS")
@@
 		(descr "SMD pad as test Point, diameter 1.0mm")
 		(tags "test point SMD pad")
-		(property "Reference" "SCK"
+		(property "Reference" "TP1"
 			(at 0 -1.448 0)
 			(layer "F.SilkS")
@@
 		(descr "SMD pad as test Point, diameter 1.0mm")
 		(tags "test point SMD pad")
-		(property "Reference" "GND"
+		(property "Reference" "TP4"
 			(at 0 -1.448 0)
 			(layer "F.SilkS")
@@
 		(descr "SMD pad as test Point, diameter 1.0mm")
 		(tags "test point SMD pad")
-		(property "Reference" "SWD"
+		(property "Reference" "TP2"
 			(at 0 -1.448 0)
 			(layer "F.SilkS")
@@
 	(footprint "extra-symbols-footprints:L0402"
 		(layer "F.Cu")
-		(at 138.57 129)
+		(at 138.45 127)
 		(property "Reference" "L3"
 			(at 0 -1.5 0)
@@
 			(size 0.79 0.54)
 			(layers "F.Cu" "F.Mask" "F.Paste")
-			(net 1 "Net-(AE1-PCB_Trace)")
+			(net 1 "Net-(AE1-FEED)")
 			(pinfunction "1")
 			(pintype "passive")
@@
 			(size 0.5 0.5)
 			(layers "F.Cu")
-			(net 2 "GND")
+			(net 1 "Net-(AE1-FEED)")
 			(pinfunction "FEED")
 			(pintype "input")
@@
 			(layers "*.Cu")
 			(remove_unused_layers no)
-			(net 1 "Net-(AE1-PCB_Trace)")
+			(net 2 "GND")
 			(pinfunction "PCB_Trace")
 			(pintype "passive")
@@
 	)
 	(segment
-		(start 136.29 127.15)
-		(end 138.14 129)
+		(start 137.575 127)
+		(end 135.625 125.05)
 		(width 0.2)
 		(layer "F.Cu")
@@
 	)
 	(segment
-		(start 135.625 127.15)
-		(end 136.29 127.15)
+		(start 137.9 127)
+		(end 137.575 127)
 		(width 0.2)
 		(layer "F.Cu")
@@
 	)
 	(segment
-		(start 140.001 127.399)
-		(end 142.601 127.399)
-		(width 0.2)
-		(layer "F.Cu")
-		(net 2)
-	)
-	(segment
 		(start 159.5 103.899)
 		(end 158.101 103.899)
@@
 	)
 	(segment
-		(start 135.625 125.05)
-		(end 137.652 125.05)
-		(width 0.2)
-		(layer "F.Cu")
-		(net 2)
-	)
-	(segment
 		(start 161.5 99.6)
 		(end 161.5 101.5)
@@
 	)
 	(segment
-		(start 137.652 125.05)
-		(end 140.001 127.399)
-		(width 0.2)
-		(layer "F.Cu")
-		(net 2)
-	)
-	(segment
 		(start 155.4 94.6)
 		(end 156.1 93.9)
@@
 	)
 	(segment
+		(start 135.625 127.15)
+		(end 139.125 130.65)
+		(width 0.2)
+		(layer "F.Cu")
+		(net 2)
+	)
+	(segment
 		(start 146.315 100.685)
 		(end 145.685 100.685)
@@
 	)
 	(segment
-		(start 142.601 127.399)
-		(end 144 126)
+		(start 139.125 130.65)
+		(end 142.55 130.65)
 		(width 0.2)
 		(layer "F.Cu")
@@
 	)
 	(segment
-		(start 141 129)
-		(end 139 129)
+		(start 155.4 117)
+		(end 155 117)
 		(width 0.2)
 		(layer "F.Cu")
@@
 	)
 	(segment
-		(start 155.4 117)
-		(end 155 117)
+		(start 155.5 115.5)
+		(end 155.5 116.9)
 		(width 0.2)
 		(layer "F.Cu")
@@
 	)
 	(segment
-		(start 155.5 115.5)
-		(end 155.5 116.9)
+		(start 139 127)
+		(end 141 129)
 		(width 0.2)
 		(layer "F.Cu")
